File: devices/KiCad/toytalk_demo_v1/toytalk_demo_v1/toytalk_demo_v1.kicad_sch (KiCad schematic)
At the start: 0 parts

Commit message: Add PCB layout and manufacturing files for ToyTalk demo v1
- Complete PCB layout in toytalk_demo_v1.kicad_pcb
- Add component libraries (INMP441 microphone, MAX98357A amp)
- Include custom KiCad parts and footprints
- Add production files for JLCPCB manufacturing
- Update project icon (icon4.png)

🤖 Generated with [Claude Code](https://claude.com/claude-code)

Co-Authored-By: Claude Sonnet 4.5 <noreply@anthropic.com>
Parts:
- added M1: INMP441, Library:INMP441_OMNIDIRECTIONAL_MICROPHONE_MODULE, symbol inmp441:INMP441_Microphone_I2S
- added U1: XIAO-ESP32-S3-DIP, Seeed:XIAO-ESP32S3-DIP, symbol Seeed:XIAO-ESP32-S3-DIP
- added U2: Max98357A, Library:MAX98357-MODULE SMD FOOTPRINT, symbol MAX98357A:Max98357
Connections:
- new net: M1.1 (L/R), M1.6 (GND), U1.13 (GND), U2.6 (GND)
- new net: M1.2 (WS), U1.3 (GPIO3/D2/A2), U2.1 (LRC)
- new net: M1.3 (SCK), U1.4 (GPIO4/D3/A3), U2.2 (BCLK)
- new net: M1.4 (SD), U1.11 (GPIO9/D10/A10/MOSI)
- new net: M1.5 (VDD), U1.12 (VCC_3V3)
- new net: U1.5 (GPIO5/D4/I2C_SDA), U2.3 (DIN)
- new net: U1.14 (VBUS), U2.4 (GAIN), U2.7 (VIN)
- new net: U1.6 (GPIO9/D5/I2C_SCL), U2.5 (SD)
