File: devices/KiCad/toytalk_demo_v3/toytalk_demo_v3.kicad_pcb (KiCad board)
At the start: 2 copper layers, 55 x 55 mm, 42 parts, among them J1 TYPE-C-31-M-12, J2 Conn_01x02, U1 ESP32-S3-WROOM-1-N8R8, U2 MAX98357AEWL_T, U3 BQ24074RGTR, U4 AP2112K-3.3TRG1, U5 TPS61022RWUR

Commit message: KiCADの回路図とPCB図を修正して再発注
Co-Authored-By: Claude Opus 4.5 <noreply@anthropic.com>
Parts:
- added C12: 10uF, Capacitor_SMD:C_0603_1608Metric, F.Cu at (64.0, 14.8)
- added S3: SKRPABE010, footprints:SW_SKRPABE010, F.Cu at (37.4, 28.6)
- moved C4 2.03 mm to (38.1, 24.5), turned to 90 degrees
Connections:
- U1 pad 13: unconnected-(U1-IO19-Pad13) -> /GPIO19
- U1 pad 14: unconnected-(U1-IO20-Pad14) -> /GPIO20
- U1 pad 19: /GPIO19 -> unconnected-(U1-IO11-Pad19)
- U1 pad 20: /GPIO20 -> unconnected-(U1-IO12-Pad20)
- U1 pad 27: unconnected-(U1-IO0-Pad27) -> /GPIO27
Routing:
- net /GPIO27: track 0.00 -> 16.3 mm
- net /GPIO19: track 51.2 -> 61.8 mm
- net /GPIO20: track 46.6 -> 56.4 mm
- net GND: track 75.4 -> 79.9 mm, vias 26 -> 29
- net /GPIO8: track 41.8 -> 44.5 mm
- net /GPIO7: track 59.2 -> 61.0 mm
- net /GPIO6: track 66.6 -> 68.3 mm
- net /+3V3: track 98.4 -> 97.0 mm
- net /GPIO3: track 72.1 -> 70.8 mm
- net unconnected-(U1-IO12-Pad20): track 0.00 -> 0.53 mm
- net Net-(U1-EN): vias 3 -> 2
