File: devices/KiCad/toytalk_demo_v3/toytalk_demo_v3.kicad_sch (KiCad schematic)
At the start: 33 parts, among them J1 TYPE-C-31-M-12, J2 Conn_01x02, U1 ESP32-S3-WROOM-1-N8R8, U2 MAX98357AEWL_T, U3 BQ24074RGTR, U4 AP2112K-3.3TRG1, U5 TPS61022RWUR

Commit message: KiCADの回路図とPCB図を修正して再発注
Co-Authored-By: Claude Opus 4.5 <noreply@anthropic.com>
Parts:
- added C12: 10uF, Capacitor_SMD:C_0603_1608Metric, symbol Device:C
- added S3: SKRPABE010, footprints:SW_SKRPABE010, symbol SKRPABE010:SKRPABE010
Connections:
- net GND: now also C12.2, S3.3, S3.4
- net GPIO19: now also U1.13 (IO19); no longer U1.19 (IO11)
- net GPIO20: now also U1.14 (IO20); no longer U1.20 (IO12)
- net VBAT: now also C12.1
- net GPIO27: now reaches U1.27 (IO0)
- net GPIO27: now also S3.1, S3.2
- no-connect marks 0 -> 33
Other:
- moved on the sheet: R4
