File: devices/KiCad/toytalker_mini_v0.2/toytalker_mini_v0.2.kicad_sch (KiCad schematic)
At the start: 28 parts, among them J1 TYPE-C-31-M-12, J2 SM02B-SRSS-TB(LF)(SN), U1 BQ25185DLHR, U2 AP2112K-3.3TRG1, U3 ESP32-S3-MINI-1-N4R2, U4 MAX98357AEWL_T

Commit message: Migrate v0.2 schematic to current KiCad file format
Opening the project with a newer KiCad rewrote toytalker_mini_v0.2.kicad_sch
into format version 20260306 (was 20250114/KiCad 9.0). No design changes:
symbol/label counts are identical. Committing so future diffs show only
real schematic edits.

Co-Authored-By: Claude Fable 5 <noreply@anthropic.com>
Parts:
- added J2: SM02B-SRSS-TB(LF)(SN), footprints:SM02B-SRSS-TB_LF__SN_, symbol SM02B-SRSS-TB_LF__SN_:SM02B-SRSS-TB_LF__SN_
- MK1: DESCRIPTION Mic Mems Digital I2s Omni -26db -> (none)
- S3: DESCRIPTION Tactile Switch SPST-NO Top Actuated Surface Mount -> (none)
- SP1: renamed from J2; DESCRIPTION SH Series 2 Position 1 mm Pitch Surface Mount Side Entry Sh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 -> (none)
Connections:
- net GND: now also J2.2; no longer SP1.2
- net VBAT: now also J2.1; no longer SP1.1
